Commit message: 수영 커밋

File: bullet/urdf/spotmicroai_sample.urdf (robot description, URDF)
Before this commit: robot SpotMicroAI, 23 links, 22 joints
Links:
- link base_link: geometry collision box size=0.14 0.11 0.07; visual box size=0.25 0.1 0.07
- link rear_link: geometry collision box size=0.04 0.11 0.07; visual box size=0.04 0.11 0.07
